Commit message: Update: Realistic URDF with battery/circuits, refined transformation logic, and stabilized OP3 walking engine

File: solidworks_export/urdf/biped_bike_robot_ver4.urdf (robot description, URDF)
Before this commit: robot biped_bike_robot_ver3, 21 links, 20 joints
Links:
- link arm_base_yaw: geometry collision mesh filename=package://biped_bike_robot_ver4/meshes/arm_base_yaw.STL; visual mesh filename=package://biped_bike_robot_ver4/meshes/arm_base_yaw.STL
- link arm_elbow_pitch: geometry collision mesh filename=package://biped_bike_robot_ver4/meshes/arm_elbow_pitch.STL; visual mesh filename=package://biped_bike_robot_ver4/meshes/arm_elbow_pitch.STL
- link arm_shoulder_pitch: mass 0.091736 -> 0.10059; geometry collision mesh filename=package://biped_bike_robot_ver4/meshes/arm_shoulder_pitch.S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; visual mesh filename=package://biped_bike_robot_ver4/meshes/arm_shoulder_pitch.S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
- link arm_wheel_pitch_: geometry collision mesh filename=package://biped_bike_robot_ver4/meshes/arm_wheel_pitch_.STL; visual mesh filename=package://biped_bike_robot_ver4/meshes/arm_wheel_pitch_.STL
- link arm_wrist_pitch: geometry collision mesh filename=package://biped_bike_robot_ver4/meshes/arm_wrist_pitch.STL; visual mesh filename=package://biped_bike_robot_ver4/meshes/arm_wrist_pitch.STL
- link arm_wrist_roll: geometry collision mesh filename=package://biped_bike_robot_ver4/meshes/arm_wrist_roll.STL; visual mesh filename=package://biped_bike_robot_ver4/meshes/arm_wrist_roll.STL
- link base_link: mass 0.20217 -> 0.55964; geometry collision mesh filename=package://biped_bike_robot_ver4/meshes/base_link.STL; visual mesh filename=package://biped_bike_robot_ver4/meshes/base_link.STL
- link l_ankle_pitch: mass 0.11708 -> 0.11682; geometry collision mesh filename=package://biped_bike_robot_ver4/meshes/l_ankle_pitch.STL; visual mesh filename=package://biped_bike_robot_ver4/meshes/l_ankle_pitch.STL
- link l_foot_roll: mass 0.073461 -> 0.074674; geometry collision mesh filename=package://biped_bike_robot_ver4/meshes/l_foot_roll.STL; visual mesh filename=package://biped_bike_robot_ver4/meshes/l_foot_roll.STL
- link l_hip_pitch: mass 0.016365 -> 0.014036; geometry collision mesh filename=package://biped_bike_robot_ver4/meshes/l_hip_pitch.STL; visual mesh filename=package://biped_bike_robot_ver4/meshes/l_hip_pitch.STL
- link l_hip_roll: mass 0.11708 -> 0.11682; geometry collision mesh filename=package://biped_bike_robot_ver4/meshes/l_hip_roll.STL; visual mesh filename=package://biped_bike_robot_ver4/meshes/l_hip_roll.STL
- link l_hip_yaw: mass 0.027291 -> 0.027149; geometry collision mesh filename=package://biped_bike_robot_ver4/meshes/l_hip_yaw.STL; visual mesh filename=package://biped_bike_robot_ver4/meshes/l_hip_yaw.STL
- link l_knee_pitch: mass 0.14474 -> 0.14522; geometry collision mesh filename=package://biped_bike_robot_ver4/meshes/l_knee_pitch.STL; visual mesh filename=package://biped_bike_robot_ver4/meshes/l_knee_pitch.STL
- link l_knee_pitch_wheel: geometry collision mesh filename=package://biped_bike_robot_ver4/meshes/l_knee_pitch_wheel.S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; visual mesh filename=package://biped_bike_robot_ver4/meshes/l_knee_pitch_wheel.S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
- link r_ankle_pitch: mass 0.11708 -> 0.11682; geometry collision mesh filename=package://biped_bike_robot_ver4/meshes/r_ankle_pitch.STL; visual mesh filename=package://biped_bike_robot_ver4/meshes/r_ankle_pitch.STL
- link r_foot_roll: mass 0.073461 -> 0.074674; geometry collision mesh filename=package://biped_bike_robot_ver4/meshes/r_foot_roll.STL; visual mesh filename=package://biped_bike_robot_ver4/meshes/r_foot_roll.STL
- link r_hip_pitch: mass 0.016365 -> 0.014036; geometry collision mesh filename=package://biped_bike_robot_ver4/meshes/r_hip_pitch.STL; visual mesh filename=package://biped_bike_robot_ver4/meshes/r_hip_pitch.STL
- link r_hip_roll: mass 0.11708 -> 0.11682; geometry collision mesh filename=package://biped_bike_robot_ver4/meshes/r_hip_roll.STL; visual mesh filename=package://biped_bike_robot_ver4/meshes/r_hip_roll.STL
- link r_hip_yaw: mass 0.027291 -> 0.027149; geometry collision mesh filename=package://biped_bike_robot_ver4/meshes/r_hip_yaw.STL; visual mesh filename=package://biped_bike_robot_ver4/meshes/r_hip_yaw.STL
- link r_knee_pitch: mass 0.14474 -> 0.14522; geometry collision mesh filename=package://biped_bike_robot_ver4/meshes/r_knee_pitch.STL; visual mesh filename=package://biped_bike_robot_ver4/meshes/r_knee_pitch.STL
- link r_knee_pitch_wheel: geometry collision mesh filename=package://biped_bike_robot_ver4/meshes/r_knee_pitch_wheel.S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; visual mesh filename=package://biped_bike_robot_ver4/meshes/r_knee_pitch_wheel.S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
Joints:
- joint arm_wheel_pitch_: origin xyz=-0.1835 0 -0.02585 rpy=0 0 0 -> xyz=-0.1865 0 -0.02595 rpy=0 0 0

File: urdf/biped_bike_robot.urdf (robot description, URDF)
Before this commit: robot biped_bike_robot_ver3, 21 links, 20 joints
Links:
- link arm_shoulder_pitch: mass 0.091736 -> 0.10059
- link base_link: mass 0.20217 -> 0.55964
- link l_ankle_pitch: mass 0.11708 -> 0.11682
- link l_foot_roll: mass 0.073461 -> 0.074674
- link l_hip_pitch: mass 0.016365 -> 0.014036
- link l_hip_roll: mass 0.11708 -> 0.11682
- link l_hip_yaw: mass 0.027291 -> 0.027149
- link l_knee_pitch: mass 0.14474 -> 0.14522
- link r_ankle_pitch: mass 0.11708 -> 0.11682
- link r_foot_roll: mass 0.073461 -> 0.074674
- link r_hip_pitch: mass 0.016365 -> 0.014036
- link r_hip_roll: mass 0.11708 -> 0.11682
- link r_hip_yaw: mass 0.027291 -> 0.027149
- link r_knee_pitch: mass 0.14474 -> 0.14522
Joints:
- joint arm_wheel_pitch__jnt: origin xyz=-0.1835 0 -0.02585 rpy=0 0 0 -> xyz=-0.1865 0 -0.02595 rpy=0 0 0
