Commit message: Update robot and configuration and transform logic

File: solidworks_export/urdf/biped_bike_robot_print_ver6.urdf (robot description, URDF)
Before this commit: robot biped_bike_robot_ver5, 20 links, 19 joints
Links:
- link arm_base_yaw: geometry collision mesh filename=package://biped_bike_robot_print_ver6/meshes/arm_base_yaw.S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; visual mesh filename=package://biped_bike_robot_print_ver6/meshes/arm_base_yaw.S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
- link arm_elbow_pitch: geometry collision mesh filename=package://biped_bike_robot_print_ver6/meshes/arm_elbow_pitc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; visual mesh filename=package://biped_bike_robot_print_ver6/meshes/arm_elbow_pitc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
- link arm_shoulder_pitch: mass 0.10092 -> 0.10542; geometry collision mesh filename=package://biped_bike_robot_print_ver6/meshes/arm_shoulder_p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; visual mesh filename=package://biped_bike_robot_print_ver6/meshes/arm_shoulder_p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
- link arm_wrist_pitch: geometry collision mesh filename=package://biped_bike_robot_print_ver6/meshes/arm_wrist_pitc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; visual mesh filename=package://biped_bike_robot_print_ver6/meshes/arm_wrist_pitc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
- link arm_wrist_roll: geometry collision mesh filename=package://biped_bike_robot_print_ver6/meshes/arm_wrist_roll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; visual mesh filename=package://biped_bike_robot_print_ver6/meshes/arm_wrist_roll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
- link base_link: mass 0.63285 -> 0.62617; geometry collision mesh filename=package://biped_bike_robot_print_ver6/meshes/base_link.STL; visual mesh filename=package://biped_bike_robot_print_ver6/meshes/base_link.STL
- link l_ankle_pitch: geometry collision mesh filename=package://biped_bike_robot_print_ver6/meshes/l_ankle_pitch.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; visual mesh filename=package://biped_bike_robot_print_ver6/meshes/l_ankle_pitch.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
- link l_foot_roll: geometry collision mesh filename=package://biped_bike_robot_print_ver6/meshes/l_foot_roll.STL; visual mesh filename=package://biped_bike_robot_print_ver6/meshes/l_foot_roll.STL
- link l_hip_pitch: geometry collision mesh filename=package://biped_bike_robot_print_ver6/meshes/l_hip_pitch.STL; visual mesh filename=package://biped_bike_robot_print_ver6/meshes/l_hip_pitch.STL
- link l_hip_roll: geometry collision mesh filename=package://biped_bike_robot_print_ver6/meshes/l_hip_roll.STL; visual mesh filename=package://biped_bike_robot_print_ver6/meshes/l_hip_roll.STL
- link l_hip_yaw: geometry collision mesh filename=package://biped_bike_robot_print_ver6/meshes/l_hip_yaw.STL; visual mesh filename=package://biped_bike_robot_print_ver6/meshes/l_hip_yaw.STL
- link l_knee_pitch: geometry collision mesh filename=package://biped_bike_robot_print_ver6/meshes/l_knee_pitch.S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; visual mesh filename=package://biped_bike_robot_print_ver6/meshes/l_knee_pitch.S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
- link l_knee_pitch_wheel: geometry collision mesh filename=package://biped_bike_robot_print_ver6/meshes/l_knee_pitch_w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; visual mesh filename=package://biped_bike_robot_print_ver6/meshes/l_knee_pitch_w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
- link r_ankle_pitch: geometry collision mesh filename=package://biped_bike_robot_print_ver6/meshes/r_ankle_pitch.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; visual mesh filename=package://biped_bike_robot_print_ver6/meshes/r_ankle_pitch.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
- link r_foot_roll: geometry collision mesh filename=package://biped_bike_robot_print_ver6/meshes/r_foot_roll.STL; visual mesh filename=package://biped_bike_robot_print_ver6/meshes/r_foot_roll.STL
- link r_hip_pitch: geometry collision mesh filename=package://biped_bike_robot_print_ver6/meshes/r_hip_pitch.STL; visual mesh filename=package://biped_bike_robot_print_ver6/meshes/r_hip_pitch.STL
- link r_hip_roll: geometry collision mesh filename=package://biped_bike_robot_print_ver6/meshes/r_hip_roll.STL; visual mesh filename=package://biped_bike_robot_print_ver6/meshes/r_hip_roll.STL
- link r_hip_yaw: geometry collision mesh filename=package://biped_bike_robot_print_ver6/meshes/r_hip_yaw.STL; visual mesh filename=package://biped_bike_robot_print_ver6/meshes/r_hip_yaw.STL
- link r_knee_pitch: geometry collision mesh filename=package://biped_bike_robot_print_ver6/meshes/r_knee_pitch.S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; visual mesh filename=package://biped_bike_robot_print_ver6/meshes/r_knee_pitch.S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
- link r_knee_pitch_wheel: geometry collision mesh filename=package://biped_bike_robot_print_ver6/meshes/r_knee_pitch_w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; visual mesh filename=package://biped_bike_robot_print_ver6/meshes/r_knee_pitch_w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
Joints:
- joint arm_elbow_pitch: origin xyz=-0.092132 -0.077697 0.0002 rpy=0 0 0.34907 -> xyz=0.0415 -0.11315 0.0002 rpy=0 0 1.5708
- joint arm_wrist_roll: axis 0.34202 0 -0.93969 -> 1 0 0; origin xyz=0.0432 -0.015 -0.0147 rpy=-1.5708 0 -1.9199 -> xyz=0.0432 -0.015 -0.0147 rpy=-1.5708 0 3.1416

File: urdf/biped_bike_robot.urdf (robot description, URDF)
Before this commit: robot biped_bike_robot_ver5, 20 links, 19 joints
Links:
- link arm_shoulder_pitch: mass 0.10092 -> 0.10542
- link base_link: mass 0.63285 -> 0.62617
Joints:
- joint arm_elbow_pitch_jnt: origin xyz=-0.092132 -0.077697 0.0002 rpy=0 0 0.34907 -> xyz=0.0415 -0.11315 0.0002 rpy=0 0 1.5708
- joint arm_shoulder_pitch_jnt: limit lower=-0.436332 upper=3.14159 effort=4.1 velocity=6.38 -> lower=-2.0944 upper=3.14159 effort=4.1 velocity=6.38
- joint arm_wrist_roll_jnt: axis 0.34202 0 -0.93969 -> 1 0 0; origin xyz=0.0432 -0.015 -0.0147 rpy=-1.5708 0 -1.9199 -> xyz=0.0432 -0.015 -0.0147 rpy=-1.5708 0 3.1416
