Commit message: feat: complete bipedal-to-3wheeled transformation sequence in simulation

File: urdf/biped_bike_robot.urdf (robot description, URDF)
Before this commit: robot biped_bike_robot_ver2, 18 links, 17 joints
Links:
- removed link arm_link_1
- removed link arm_link_2
- removed link elbow_wheel
- removed link end_effector
- removed link l_ankle_joint
- removed link l_foot_link
- removed link l_hip_pitch_joint
- removed link l_hip_roll_joint
- removed link l_knee_joint
- removed link l_knee_wheel
- removed link r_ankle_joint
- removed link r_foot_link
- removed link r_hip_pitch_link
- removed link r_hip_roll_joint
- removed link r_knee_joint
- removed link r_knee_wheel
- removed link waist_yaw_link
- added link arm_base_yaw, mass 0.052551; collision mesh filename=package://biped_bike_robot/meshes/arm_base_yaw.STL; visual mesh filename=package://biped_bike_robot/meshes/arm_base_yaw.STL
- added link arm_elbow_pitch, mass 0.046725; collision mesh filename=package://biped_bike_robot/meshes/arm_elbow_pitch.STL; visual mesh filename=package://biped_bike_robot/meshes/arm_elbow_pitch.STL
- added link arm_shoulder_pitch, mass 0.091736; collision mesh filename=package://biped_bike_robot/meshes/arm_shoulder_pitch.STL; visual mesh filename=package://biped_bike_robot/meshes/arm_shoulder_pitch.STL
- added link arm_wheel_pitch_, mass 0.012433; collision mesh filename=package://biped_bike_robot/meshes/arm_wheel_pitch_.STL; visual mesh filename=package://biped_bike_robot/meshes/arm_wheel_pitch_.STL
- added link arm_wrist_pitch, mass 0.019754; collision mesh filename=package://biped_bike_robot/meshes/arm_wrist_pitch.STL; visual mesh filename=package://biped_bike_robot/meshes/arm_wrist_pitch.STL
- added link arm_wrist_roll, mass 0.039491; collision mesh filename=package://biped_bike_robot/meshes/arm_wrist_roll.STL; visual mesh filename=package://biped_bike_robot/meshes/arm_wrist_roll.STL
- added link l_ankle_pitch, mass 0.11708; collision mesh filename=package://biped_bike_robot/meshes/l_ankle_pitch.STL; visual mesh filename=package://biped_bike_robot/meshes/l_ankle_pitch.STL
- added link l_foot_roll, mass 0.073461; collision mesh filename=package://biped_bike_robot/meshes/l_foot_roll.STL; visual mesh filename=package://biped_bike_robot/meshes/l_foot_roll.STL
- added link l_hip_pitch, mass 0.016365; collision mesh filename=package://biped_bike_robot/meshes/l_hip_pitch.STL; visual mesh filename=package://biped_bike_robot/meshes/l_hip_pitch.STL
- added link l_hip_roll, mass 0.11708; collision mesh filename=package://biped_bike_robot/meshes/l_hip_roll.STL; visual mesh filename=package://biped_bike_robot/meshes/l_hip_roll.STL
- added link l_hip_yaw, mass 0.027291; collision mesh filename=package://biped_bike_robot/meshes/l_hip_yaw.STL; visual mesh filename=package://biped_bike_robot/meshes/l_hip_yaw.STL
- added link l_knee_pitch, mass 0.14474; collision mesh filename=package://biped_bike_robot/meshes/l_knee_pitch.STL; visual mesh filename=package://biped_bike_robot/meshes/l_knee_pitch.STL
- added link l_knee_pitch_wheel, mass 0.012433; collision mesh filename=package://biped_bike_robot/meshes/l_knee_pitch_wheel.STL; visual mesh filename=package://biped_bike_robot/meshes/l_knee_pitch_wheel.STL
- added link r_ankle_pitch, mass 0.11708; collision mesh filename=package://biped_bike_robot/meshes/r_ankle_pitch.STL; visual mesh filename=package://biped_bike_robot/meshes/r_ankle_pitch.STL
- added link r_foot_roll, mass 0.073461; collision mesh filename=package://biped_bike_robot/meshes/r_foot_roll.STL; visual mesh filename=package://biped_bike_robot/meshes/r_foot_roll.STL
- added link r_hip_pitch, mass 0.016365; collision mesh filename=package://biped_bike_robot/meshes/r_hip_pitch.STL; visual mesh filename=package://biped_bike_robot/meshes/r_hip_pitch.STL
- added link r_hip_roll, mass 0.11708; collision mesh filename=package://biped_bike_robot/meshes/r_hip_roll.STL; visual mesh filename=package://biped_bike_robot/meshes/r_hip_roll.STL
- added link r_hip_yaw, mass 0.027291; collision mesh filename=package://biped_bike_robot/meshes/r_hip_yaw.STL; visual mesh filename=package://biped_bike_robot/meshes/r_hip_yaw.STL
- added link r_knee_pitch, mass 0.14474; collision mesh filename=package://biped_bike_robot/meshes/r_knee_pitch.STL; visual mesh filename=package://biped_bike_robot/meshes/r_knee_pitch.STL
- added link r_knee_pitch_wheel, mass 0.012433; collision mesh filename=package://biped_bike_robot/meshes/r_knee_pitch_wheel.STL; visual mesh filename=package://biped_bike_robot/meshes/r_knee_pitch_wheel.STL
- link base_link: mass 0.14124 -> 0.20217
Joints:
- removed joint arm_link_1_jnt_jnt
- removed joint arm_link_2_jnt_jnt
- removed joint elbow_wheel_jnt_jnt
- removed joint end_effector_jnt_jnt
- removed joint l_ankle_joint_jnt_jnt
- removed joint l_foot_link_jnt_jnt
- removed joint l_hip_pitch_joint_jnt_jnt
- removed joint l_hip_roll_joint_jnt_jnt
- removed joint l_knee_joint_jnt_jnt
- removed joint l_knee_wheel_jnt_jnt
- removed joint r_ankle_joint_jnt_jnt
- removed joint r_foot_link_jnt_jnt
- removed joint r_hip_pitch_link_jnt_jnt
- removed joint r_hip_roll_joint_jnt_jnt
- removed joint r_knee_joint_jnt_jnt
- removed joint r_knee_wheel_jnt_jnt
- removed joint waist_yaw_link_jnt_jnt
- added joint arm_base_yaw_jnt: type revolute, parent base_link, child arm_base_yaw, origin xyz=-0.01505 -0.07695 0.0444 rpy=0 0 0, axis 0 0 -1, limit lower=-3.14159 upper=3.14159 effort=1.5 velocity=6.38
- added joint arm_elbow_pitch_jnt: type revolute, parent arm_shoulder_pitch, child arm_elbow_pitch, origin xyz=-0.11295 -0.0415 0 rpy=0 0 0, axis 0 0 1, limit lower=-3.14159 upper=3.14159 effort=1.5 velocity=6.38
- added joint arm_shoulder_pitch_jnt: type revolute, parent arm_base_yaw, child arm_shoulder_pitch, origin xyz=-0.0002 0.0209 0.04235 rpy=-1.5708 0 0, axis 0 0 1, limit lower=-3.14159 upper=3.14159 effort=1.5 velocity=6.38
- added joint arm_wheel_pitch__jnt: type continuous, parent arm_shoulder_pitch, child arm_wheel_pitch_, origin xyz=-0.1835 0 -0.02585 rpy=0 0 0, axis 0 0 -1, limit effort=1.5 velocity=6.38
- added joint arm_wrist_pitch_jnt: type revolute, parent arm_elbow_pitch, child arm_wrist_pitch, origin xyz=0.1618 0 -0.0064 rpy=0 0 0, axis 0 0 -1, limit lower=-3.14159 upper=3.14159 effort=1.5 velocity=6.38
- added joint arm_wrist_roll_jnt: type revolute, parent arm_wrist_pitch, child arm_wrist_roll, origin xyz=0.0432 -0.015 -0.0147 rpy=-1.5708 0 -1.5708, axis 0 0 -1, limit lower=-3.14159 upper=3.14159 effort=1.5 velocity=6.38
- added joint l_ankle_pitch_jnt: type revolute, parent l_knee_pitch, child l_ankle_pitch, origin xyz=0 0.08775 0 rpy=0 0 0, axis 0 0 -1, limit lower=-3.14159 upper=3.14159 effort=1.5 velocity=6.38
- added joint l_foot_roll_jnt: type revolute, parent l_ankle_pitch, child l_foot_roll, origin xyz=-0.0614 0 -0.0209 rpy=-1.5708 0 -1.5708, axis 0 0 -1, limit lower=-3.14159 upper=3.14159 effort=1.5 velocity=6.38
- added joint l_hip_pitch_jnt: type revolute, parent l_hip_roll, child l_hip_pitch, origin xyz=-0.024 -0.0209 0.0614 rpy=1.5708 -1.5708 0, axis 0 0 1, limit lower=-3.14159 upper=3.14159 effort=1.5 velocity=6.38
- added joint l_hip_roll_jnt: type revolute, parent l_hip_yaw, child l_hip_roll, origin xyz=-0.0614 0 -0.0356 rpy=0 -1.5708 3.14159, axis 0 0 -1, limit lower=-3.14159 upper=3.14159 effort=1.5 velocity=6.38
- added joint l_hip_yaw_jnt: type revolute, parent base_link, child l_hip_yaw, origin xyz=-0.01525 -0.01425 0.0026 rpy=0 0 0, axis 0 0 -1, limit lower=-3.14159 upper=3.14159 effort=1.5 velocity=6.38
- added joint l_knee_pitch_jnt: type revolute, parent l_hip_pitch, child l_knee_pitch, origin xyz=0 0.059 0 rpy=0 0 0, axis 0 0 -1, limit lower=-3.14159 upper=3.14159 effort=1.5 velocity=6.38
- added joint l_knee_pitch_wheel_jnt: type continuous, parent l_knee_pitch, child l_knee_pitch_wheel, origin xyz=0.047 0.024 0 rpy=0 0 0, axis 0 0 -1, limit effort=1.5 velocity=6.38
- added joint r_ankle_pitch_jnt: type revolute, parent r_knee_pitch, child r_ankle_pitch, origin xyz=0 0.08775 0 rpy=0 0 0, axis 0 0 -1, limit lower=-3.14159 upper=3.14159 effort=1.5 velocity=6.38
- added joint r_foot_roll_jnt: type revolute, parent r_ankle_pitch, child r_foot_roll, origin xyz=-0.0614 0 -0.0209 rpy=-1.5708 0 -1.5708, axis 0 0 -1, limit lower=-3.14159 upper=3.14159 effort=1.5 velocity=6.38
- added joint r_hip_pitch_jnt: type revolute, parent r_hip_roll, child r_hip_pitch, origin xyz=-0.024 -0.0209 0.0614 rpy=1.5708 -1.5708 0, axis 0 0 -1, limit lower=-3.14159 upper=3.14159 effort=1.5 velocity=6.38
- added joint r_hip_roll_jnt: type revolute, parent r_hip_yaw, child r_hip_roll, origin xyz=-0.0614 0 -0.0356 rpy=0 -1.5708 3.14159, axis 0 0 -1, limit lower=-3.14159 upper=3.14159 effort=1.5 velocity=6.38
- added joint r_hip_yaw_jnt: type revolute, parent base_link, child r_hip_yaw, origin xyz=-0.01525 -0.13925 0.0026 rpy=0 0 0, axis 0 0 -1, limit lower=-3.14159 upper=3.14159 effort=1.5 velocity=6.38
- added joint r_knee_pitch_jnt: type revolute, parent r_hip_pitch, child r_knee_pitch, origin xyz=0 0.059 0 rpy=0 0 0, axis 0 0 -1, limit lower=-3.14159 upper=3.14159 effort=1.5 velocity=6.38
- added joint r_knee_pitch_wheel_jnt: type continuous, parent r_knee_pitch, child r_knee_pitch_wheel, origin xyz=0.047 0.024 0 rpy=0 0 0, axis 0 0 1, limit effort=1.5 velocity=6.38

Commit message: feat: 실물 동작 안정화 및 바이크 휠 키보드 제어 추가

File: urdf/biped_bike_robot.urdf (robot description, URDF)
Before this commit: robot biped_bike_robot_ver4, 21 links, 20 joints
Joints:
- joint arm_shoulder_pitch_jnt: limit lower=-3.14159 upper=3.14159 effort=1.5 velocity=6.38 -> lower=-0.436332 upper=3.14159 effort=1.5 velocity=6.38

Commit message: feat: update URDF v5 and add robot web interface

File: urdf/biped_bike_robot.urdf (robot description, URDF)
Before this commit: robot biped_bike_robot_ver4, 21 links, 20 joints
Links:
- removed link arm_wheel_pitch_
- link arm_elbow_pitch: mass 0.046725 -> 0.043796
- link arm_shoulder_pitch: mass 0.10059 -> 0.10092
- link base_link: mass 0.55964 -> 0.63285
- link l_ankle_pitch: mass 0.11682 -> 0.11819
- link l_foot_roll: mass 0.074674 -> 0.074723
- link l_hip_roll: mass 0.11682 -> 0.11819
- link l_hip_yaw: mass 0.027149 -> 0.02669
- link l_knee_pitch: mass 0.14522 -> 0.14629
- link l_knee_pitch_wheel: mass 0.012433 -> 0.016569
- link r_ankle_pitch: mass 0.11682 -> 0.11819
- link r_foot_roll: mass 0.074674 -> 0.074723
- link r_hip_roll: mass 0.11682 -> 0.11819
- link r_hip_yaw: mass 0.027149 -> 0.02669
- link r_knee_pitch: mass 0.14522 -> 0.14629
- link r_knee_pitch_wheel: mass 0.012433 -> 0.016569
Joints:
- removed joint arm_wheel_pitch__jnt
- joint arm_elbow_pitch_jnt: axis 0 0 1 -> 0 0 -1; origin xyz=-0.11295 -0.0415 0 rpy=0 0 0 -> xyz=-0.092132 -0.077697 0.0002 rpy=0 0 0.34907
- joint arm_shoulder_pitch_jnt: limit lower=-0.436332 upper=3.14159 effort=1.5 velocity=6.38 -> lower=-0.436332 upper=3.14159 effort=4.1 velocity=6.38
- joint arm_wrist_pitch_jnt: origin xyz=0.1618 0 -0.0064 rpy=0 0 0 -> xyz=0.14632 0 -0.006 rpy=0 0 0
- joint arm_wrist_roll_jnt: axis 0 0 -1 -> 0.34202 0 -0.93969; origin xyz=0.0432 -0.015 -0.0147 rpy=-1.5708 0 -1.5708 -> xyz=0.0432 -0.015 -0.0147 rpy=-1.5708 0 -1.9199
- joint l_ankle_pitch_jnt: origin xyz=0 0.08775 0 rpy=0 0 0 -> xyz=-0.003 0.1125 0 rpy=0 0 0
- joint l_hip_roll_jnt: origin xyz=-0.0614 0 -0.0356 rpy=0 -1.5708 3.14159 -> xyz=-0.0594 0 -0.0376 rpy=0 -1.5708 3.14159
- joint l_knee_pitch_wheel_jnt: origin xyz=0.047 0.024 0 rpy=0 0 0 -> xyz=0.041 0 0 rpy=0 0 0
- joint r_ankle_pitch_jnt: origin xyz=0 0.08775 0 rpy=0 0 0 -> xyz=-0.005 0.1125 0 rpy=0 0 0
- joint r_foot_roll_jnt: origin xyz=-0.0614 0 -0.0209 rpy=-1.5708 0 -1.5708 -> xyz=-0.0594 0.00025 -0.0209 rpy=-1.5708 0 -1.5708
- joint r_hip_roll_jnt: origin xyz=-0.0614 0 -0.0356 rpy=0 -1.5708 3.14159 -> xyz=-0.0594 0 -0.0376 rpy=0 -1.5708 3.14159
- joint r_knee_pitch_wheel_jnt: origin xyz=0.047 0.024 0 rpy=0 0 0 -> xyz=0.041 0 0 rpy=0 0 0

File: urdf/biped_bike_robot_ver5.urdf (robot description, URDF)
Before this commit: robot biped_bike_robot_ver4, 21 links, 20 joints
Links:
- removed link arm_wheel_pitch_
- link arm_base_yaw: geometry collision mesh filename=package://biped_bike_robot_ver5/meshes/arm_base_yaw.STL; visual mesh filename=package://biped_bike_robot_ver5/meshes/arm_base_yaw.STL
- link arm_elbow_pitch: mass 0.046725 -> 0.043796; geometry collision mesh filename=package://biped_bike_robot_ver5/meshes/arm_elbow_pitch.STL; visual mesh filename=package://biped_bike_robot_ver5/meshes/arm_elbow_pitch.STL
- link arm_shoulder_pitch: mass 0.10059 -> 0.10092; geometry collision mesh filename=package://biped_bike_robot_ver5/meshes/arm_shoulder_pitch.S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; visual mesh filename=package://biped_bike_robot_ver5/meshes/arm_shoulder_pitch.S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
- link arm_wrist_pitch: geometry collision mesh filename=package://biped_bike_robot_ver5/meshes/arm_wrist_pitch.STL; visual mesh filename=package://biped_bike_robot_ver5/meshes/arm_wrist_pitch.STL
- link arm_wrist_roll: geometry collision mesh filename=package://biped_bike_robot_ver5/meshes/arm_wrist_roll.STL; visual mesh filename=package://biped_bike_robot_ver5/meshes/arm_wrist_roll.STL
- link base_link: mass 0.55964 -> 0.63285; geometry collision mesh filename=package://biped_bike_robot_ver5/meshes/base_link.STL; visual mesh filename=package://biped_bike_robot_ver5/meshes/base_link.STL
- link l_ankle_pitch: mass 0.11682 -> 0.11819; geometry collision mesh filename=package://biped_bike_robot_ver5/meshes/l_ankle_pitch.STL; visual mesh filename=package://biped_bike_robot_ver5/meshes/l_ankle_pitch.STL
- link l_foot_roll: mass 0.074674 -> 0.074723; geometry collision mesh filename=package://biped_bike_robot_ver5/meshes/l_foot_roll.STL; visual mesh filename=package://biped_bike_robot_ver5/meshes/l_foot_roll.STL
- link l_hip_pitch: geometry collision mesh filename=package://biped_bike_robot_ver5/meshes/l_hip_pitch.STL; visual mesh filename=package://biped_bike_robot_ver5/meshes/l_hip_pitch.STL
- link l_hip_roll: mass 0.11682 -> 0.11819; geometry collision mesh filename=package://biped_bike_robot_ver5/meshes/l_hip_roll.STL; visual mesh filename=package://biped_bike_robot_ver5/meshes/l_hip_roll.STL
- link l_hip_yaw: mass 0.027149 -> 0.02669; geometry collision mesh filename=package://biped_bike_robot_ver5/meshes/l_hip_yaw.STL; visual mesh filename=package://biped_bike_robot_ver5/meshes/l_hip_yaw.STL
- link l_knee_pitch: mass 0.14522 -> 0.14629; geometry collision mesh filename=package://biped_bike_robot_ver5/meshes/l_knee_pitch.STL; visual mesh filename=package://biped_bike_robot_ver5/meshes/l_knee_pitch.STL
- link l_knee_pitch_wheel: mass 0.012433 -> 0.016569; geometry collision mesh filename=package://biped_bike_robot_ver5/meshes/l_knee_pitch_wheel.S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; visual mesh filename=package://biped_bike_robot_ver5/meshes/l_knee_pitch_wheel.S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
- link r_ankle_pitch: mass 0.11682 -> 0.11819; geometry collision mesh filename=package://biped_bike_robot_ver5/meshes/r_ankle_pitch.STL; visual mesh filename=package://biped_bike_robot_ver5/meshes/r_ankle_pitch.STL
- link r_foot_roll: mass 0.074674 -> 0.074723; geometry collision mesh filename=package://biped_bike_robot_ver5/meshes/r_foot_roll.STL; visual mesh filename=package://biped_bike_robot_ver5/meshes/r_foot_roll.STL
- link r_hip_pitch: geometry collision mesh filename=package://biped_bike_robot_ver5/meshes/r_hip_pitch.STL; visual mesh filename=package://biped_bike_robot_ver5/meshes/r_hip_pitch.STL
- link r_hip_roll: mass 0.11682 -> 0.11819; geometry collision mesh filename=package://biped_bike_robot_ver5/meshes/r_hip_roll.STL; visual mesh filename=package://biped_bike_robot_ver5/meshes/r_hip_roll.STL
- link r_hip_yaw: mass 0.027149 -> 0.02669; geometry collision mesh filename=package://biped_bike_robot_ver5/meshes/r_hip_yaw.STL; visual mesh filename=package://biped_bike_robot_ver5/meshes/r_hip_yaw.STL
- link r_knee_pitch: mass 0.14522 -> 0.14629; geometry collision mesh filename=package://biped_bike_robot_ver5/meshes/r_knee_pitch.STL; visual mesh filename=package://biped_bike_robot_ver5/meshes/r_knee_pitch.STL
- link r_knee_pitch_wheel: mass 0.012433 -> 0.016569; geometry collision mesh filename=package://biped_bike_robot_ver5/meshes/r_knee_pitch_wheel.S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; visual mesh filename=package://biped_bike_robot_ver5/meshes/r_knee_pitch_wheel.S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
Joints:
- removed joint arm_wheel_pitch_
- joint arm_elbow_pitch: axis 0 0 1 -> 0 0 -1; origin xyz=-0.11295 -0.0415 0 rpy=0 0 0 -> xyz=-0.092132 -0.077697 0.0002 rpy=0 0 0.34907
- joint arm_wrist_pitch: origin xyz=0.1618 0 -0.0064 rpy=0 0 0 -> xyz=0.14632 0 -0.006 rpy=0 0 0
- joint arm_wrist_roll: axis 0 0 -1 -> 0.34202 0 -0.93969; origin xyz=0.0432 -0.015 -0.0147 rpy=-1.5708 0 -1.5708 -> xyz=0.0432 -0.015 -0.0147 rpy=-1.5708 0 -1.9199
- joint l_ankle_pitch: origin xyz=0 0.08775 0 rpy=0 0 0 -> xyz=-0.003 0.1125 0 rpy=0 0 0
- joint l_hip_roll: origin xyz=-0.0614 0 -0.0356 rpy=0 -1.5708 0 -> xyz=-0.0594 0 -0.0376 rpy=0 -1.5708 0
- joint l_knee_pitch_wheel: origin xyz=0.047 0.024 0 rpy=0 0 0 -> xyz=0.041 0 0 rpy=0 0 0
- joint r_ankle_pitch: origin xyz=0 0.08775 0 rpy=0 0 0 -> xyz=-0.005 0.1125 0 rpy=0 0 0
- joint r_foot_roll: origin xyz=-0.0614 0 -0.0209 rpy=-1.5708 0 -1.5708 -> xyz=-0.0594 0.00025 -0.0209 rpy=-1.5708 0 -1.5708
- joint r_hip_roll: origin xyz=-0.0614 0 -0.0356 rpy=0 -1.5708 0 -> xyz=-0.0594 0 -0.0376 rpy=0 -1.5708 0
- joint r_knee_pitch: axis 0 0 -1 -> 0 0 1
- joint r_knee_pitch_wheel: origin xyz=0.047 0.024 0 rpy=0 0 0 -> xyz=0.041 0 0 rpy=0 0 0
