Commit message: Update bike transform and robot control

File: urdf/biped_bike_robot.urdf (robot description, URDF)
Before this commit: robot biped_bike_robot_print_ver6, 20 links, 19 joints
Joints:
- joint l_foot_roll_jnt: limit lower=-3.14159 upper=3.14159 effort=1.5 velocity=6.38 -> lower=-3.14159 upper=3.14159 effort=3.0 velocity=8.063
- joint l_knee_pitch_jnt: limit lower=-3.14159 upper=3.14159 effort=1.5 velocity=6.38 -> lower=-3.14159 upper=3.14159 effort=3.0 velocity=8.063
- joint r_foot_roll_jnt: limit lower=-3.14159 upper=3.14159 effort=1.5 velocity=6.38 -> lower=-3.14159 upper=3.14159 effort=3.0 velocity=8.063
- joint r_knee_pitch_jnt: limit lower=-3.14159 upper=3.14159 effort=1.5 velocity=6.38 -> lower=-3.14159 upper=3.14159 effort=3.0 velocity=8.063
